File: hardware/imu-to-ttl/02_mcu.kicad_sch (KiCad schematic)
At the start: 6 parts, among them J2 SWD+UART+NRST, U1 STM32G031F8P6

Commit message: sync: 2026-10-12 日常更新
Connections:
- no-connect marks 5 -> 3
Changed lines of the file:
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@@
 	)
 	)
-	(no_connect (at 74.93 107.95))
 	(no_connect (at 74.93 110.49))
 	(no_connect (at 74.93 100.33))
-	(no_connect (at 125.73 97.79))
 	(no_connect (at 74.93 105.41))
 	(text "MCU - STM32G031F8P6 (TSSOP-20)"

Commit message: sync: 2026-10-12 日常更新
Changed lines of the file:
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@@
 	)
 		(property "Value" "100nF 50V"
-		(at 59.61 154.36 0)
+		(at 46.99 154.36 0)
 		(effects
 		(font
@@
 	)
 		(property "Value" "4.7uF 10V X7R"
-		(at 85.01 154.36 0)
+		(at 72.39 154.36 0)
 		(effects
 		(font
@@
 	)
 		(property "Value" "10k"
-		(at 59.61 64.19 0)
+		(at 46.99 64.19 0)
 		(effects
 		(font
@@
 	)
 		(property "Value" "100nF 50V"
-		(at 85.01 64.19 0)
-		(effects
-		(font
+		(at 72.39 64.19 0)
+		(effects
+		(font

Commit message: sync: 2026-10-12 日常更新
Parts:
- J2: footprint Connector_PinHeader_2.54mm:PinHeader_1x07_P2.54mm_Vertical -> Connector_PinHeader_2.54mm:PinHeader_1x07_P2.54mm_Horizontal
Changed lines of the file:
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@@
 	)
 	)
-		(property "Footprint" "Connector_PinHeader_2.54mm:PinHeader_1x07_P2.54mm_Vertical"
+		(property "Footprint" "Connector_PinHeader_2.54mm:PinHeader_1x07_P2.54mm_Horizontal"
 		(at 219.71 110.49 0)
 		(effects

Commit message: sync: 2026-10-15 日常更新
Parts:
- J2: footprint Connector_PinHeader_2.54mm:PinHeader_1x07_P2.54mm_Horizontal -> Connector_PinHeader_2.54mm:PinHeader_1x07_P2.54mm_Vertical
Connections:
- net MCU_RX renamed BUS_LOGIC
- net RX_EN: no longer names the net of U1.1 (PB7/PB8)
- net TX_EN_N: no longer names the net of U1.8 (PA1)
- no-connect marks 3 -> 5

Commit message: sync: 2026-10-12 日常更新
Connections:
- net RX_EN: now reaches U1.1 (PB7/PB8)
- net TX_EN_N: now reaches U1.8 (PA1)
- net BUS_LOGIC renamed MCU_RX
Changed lines of the file:
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@@
 	)
+	)
+	(global_label "TX_EN_N"
+		(shape bidirectional)
+		(at 125.73 97.79 0)
+		(fields_autoplaced yes)
+		(effects
+			(font
+				(size 1.27 1.27)
+			)
+			(justify left)
+		)
+		(property "Intersheetrefs" "${INTERSHEET_REFS}"
+			(at 125.73 97.79 0)
+			(effects
+				(font
+					(size 1.27 1.27)
+				)
+				(hide yes)
+			)
+		)
+	)
+	(global_label "RX_EN"
+		(shape bidirectional)
+		(at 74.93 107.95 180)
+		(fields_autoplaced yes)
+		(effects
+			(font
+				(size 1.27 1.27)
+			)
+			(justify right)
+		)
+		(property "Intersheetrefs" "${INTERSHEET_REFS}"
+			(at 74.93 107.95 0)
+			(effects
+				(font
+					(size 1.27 1.27)
+				)
+				(hide yes)
+			)
+		)
 	)
 	(global_label "BUS_TX"
@@
 	)
 	)
-	(global_label "BUS_LOGIC"
+	(global_label "MCU_RX"
 		(shape bidirectional)
 		(at 125.73 102.87 0)
