File: hardware/imu-to-ttl/03_imu.kicad_sch (KiCad schematic)
At the start: 9 parts, among them U2 LSM6DSV16XTR

Commit message: sync: 2026-10-12 日常更新
Changed lines of the file:
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@@
 		(dnp no)
 		(property "Reference" "FB1"
-		(at 165.02 55.19 0)
+		(at 151.13 57.15 0)
 		(effects
 		(font
@@
 	)
 		(property "Value" "BLM18AG601SN1D"
-		(at 165.02 64.19 0)
+		(at 151.13 62.23 0)
 		(effects
 		(font
@@
 		(dnp no)
 		(property "Reference" "C10"
-		(at 165.02 75.51 0)
+		(at 151.13 77.47 0)
 		(effects
 		(font
@@
 	)
 		(property "Value" "100nF 50V"
-		(at 165.02 84.51 0)
+		(at 151.13 82.55 0)
 		(effects
 		(font
@@
 		(dnp no)
 		(property "Reference" "C11"
-		(at 165.02 90.75 0)
+		(at 151.13 92.71 0)
 		(effects
 		(font
@@
 	)
 		(property "Value" "100nF 50V"
-		(at 165.02 99.75 0)
+		(at 151.13 97.79 0)
 		(effects
 		(font
@@
 		(dnp no)
 		(property "Reference" "C12"
-		(at 165.02 105.99 0)
+		(at 151.13 107.95 0)
 		(effects
 		(font
@@
 	)
 		(property "Value" "1uF 25V X7R"
-		(at 165.02 114.99 0)
+		(at 151.13 113.03 0)
 		(effects
 		(font
@@
 	)
 		(property "Value" "10k"
-		(at 59.61 84.51 0)
+		(at 46.99 83.82 0)
 		(effects
 		(font
@@
 		(dnp no)
 		(property "Reference" "R6"
-		(at 165.02 130.12 0)
+		(at 151.13 132.08 0)
 		(effects
 		(font
@@
 	)
 		(property "Value" "0R"
-		(at 165.02 139.12 0)
-		(effects
-		(font
+		(at 151.13 137.16 0)
+		(effects
+		(font

Commit message: sync: 2026-10-12 日常更新
Other:
- note added: "SDx/SCx pull-downs (R4/R5) terminate the aux I3C bus; OCS_AUX pull-up R6 per datasheet"

Commit message: sync: 2026-10-15 日常更新
Other:
- note removed: "SDx/SCx pull-downs (R4/R5) terminate the aux I3C bus; OCS_AUX pull-up R6 per datasheet"
