File: hardware/imu-to-ttl/imu_to_ttl.kicad_pcb (KiCad board)
At the start: 2 copper layers, 41 x 30 mm, 54 parts, among them J1 BATT IN 2.54 2P, J2 SWD+UART+NRST, J3 J_NECK, J4 J_L, J5 J_R, Q1 AO4407C, U1 STM32G031F8P6, U2 LSM6DSV16XTR, U3 SN74LVC1G125DBVT, U4 HT7533-1

Commit message: sync: 2026-10-12 日常更新
Parts:
- added R14: 10k, R_0603_1608Metric, B.Cu at (33.7, 3.10)
- added R15: 10k, R_0603_1608Metric, B.Cu at (31.9, 8.00)
- added R16: 10k, R_0603_1608Metric, B.Cu at (28.5, 3.10)
- U3: value SN74LVC1G125DBVT -> SN74LVC2G241DCUR; footprint SOT-23-5 -> Package_SO:TSSOP-8_3x3mm_P0.65mm
- moved U3 0.36 mm to (32.2, 6.90)
Connections:
- U1 pad 1: unconnected-(U1-PB7/PB8-Pad1) -> RX_EN
- U1 pad 10: BUS_LOGIC -> MCU_RX
- U1 pad 8: unconnected-(U1-PA1-Pad8) -> TX_EN_N
- U3 pad 1: BUS_TX -> TX_EN_N
- U3 pad 3: GND -> MCU_RX
- U3 pad 4: BUS_LOGIC -> GND
- U3 pad 5: +3V3 -> BUS_LOGIC
Routing:
- net GND: track 162.6 -> 141.6 mm, vias 8 -> 7
- net +3V3: track 114.9 -> 101.5 mm, vias 6 -> 5
- net NRST: track 41.0 -> 28.2 mm, vias 2 -> 1
- net BUS_DATA: track 47.9 -> 35.8 mm, vias 3 -> 1
- net BUS_TX: track 43.0 -> 33.3 mm
- net BUS_CLAMP: track 19.6 -> 11.5 mm
- net BUS_LOGIC: track 27.6 -> 21.3 mm
- net SPI_MISO: track 17.9 -> 11.6 mm
- net SWCLK: track 19.9 -> 14.5 mm
- net UART1_RX: track 12.4 -> 7.81 mm
- net SPI_CS: track 24.6 -> 20.5 mm
- net SPI_SCK: track 19.5 -> 15.5 mm
- net SWDIO: track 17.1 -> 13.7 mm
- net OCS_AUX: track 11.3 -> 8.36 mm, vias 2 -> 1
- net VBAT_LOGIC: track 60.2 -> 58.3 mm
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
Commit message: sync: 2026-10-12 日常更新
Parts:
- C6, C9, R13, R2, TH1: moved to B.Cu
- J2: footprint PinHeader_1x07_P2.54mm_Vertical -> PinHeader_1x07_P2.54mm_Horizontal
- J3, J4, J5: footprint JST_PH_B3B-PH-K_1x03_P2.00mm_Vertical -> PinHeader_1x03_P2.54mm_Horizontal
- R14, R15, R16: moved to F.Cu
- U3: footprint Package_SO:TSSOP-8_3x3mm_P0.65mm -> TSSOP-8_3x3mm_P0.65mm
- moved C7 29.7 mm to (15.3, 5.28)
- moved F1 28.3 mm to (28.3, 11.5)
- moved Q1 28.0 mm to (28.8, 7.90)
- moved R2 25.9 mm to (20.5, 3.80)
- moved TH1 24.6 mm to (13.0, 25.5)
- moved R16 24.5 mm to (35.8, 26.5)
- moved C13 24.1 mm to (23.0, 4.28)
- moved R13 23.2 mm to (23.5, 28.2)
- moved C5 21.1 mm to (11.5, 4.00)
- moved U4 20.9 mm to (16.5, 5.50)
- moved R14 19.9 mm to (25.5, 21.3)
- moved J3 18.5 mm to (21.4, 25.5), turned to -90 degrees
- moved R15 18.1 mm to (26.5, 25.3)
- moved R6 17.1 mm to (15.3, 7.28)
- moved C14 16.6 mm to (20.4, 22.5), turned to 180 degrees
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Connections:
- R16 pad 1: GND -> RX_EN
- R16 pad 2: RX_EN -> GND
Routing:
- net NRST: track 28.2 -> 89.1 mm, vias 1 -> 5
- net GND: track 141.6 -> 199.5 mm, vias 7 -> 5
- net VBAT_RAW: track 14.4 -> 55.2 mm, vias 1 -> 4
- net UART1_TX: track 16.4 -> 57.2 mm, vias 0 -> 3
- net UART1_RX: track 7.81 -> 44.7 mm, vias 0 -> 4
- net SWCLK: track 14.5 -> 51.3 mm, vias 0 -> 3
- net BUS_LOGIC: track 21.3 -> 52.5 mm, vias 2 -> 1
- net BUS_CLAMP: track 11.5 -> 41.4 mm, vias 0 -> 1
- net +3V3: track 101.5 -> 129.6 mm, vias 5 -> 3
- net RX_EN: track 0.00 -> 26.8 mm, vias 0 -> 2
- net V3V3_IMU: track 74.7 -> 58.1 mm, vias 5 -> 6
- net VBAT: track 93.7 -> 79.3 mm
- net BUS_DATA: track 35.8 -> 49.1 mm, vias 1 -> 5
- net Q1_GATE: track 44.0 -> 56.6 mm
- net SPI_MISO: track 11.6 -> 23.9 mm, vias 2 -> 4
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
Commit message: sync: 2026-10-14 日常更新
Parts:
- J1: value BATT IN 2.54 2P -> BattPad_1x02_P3.6; footprint TerminalBlock_Xinya_XY308-2.54-2P_1x02_P2.54mm_Horizontal -> BattPad_1x02_P3.60mm_Drill1.2mm
- moved J1 0.20 mm to (4.40, 26.5), turned to 0 degrees
Routing:
- net Q1_GATE: track 56.6 -> 58.0 mm
- net NRST: track 89.1 -> 90.2 mm

Commit message: sync: 2026-10-15 日常更新
Parts:
- moved TH1 13.6 mm to (26.3, 28.2)
- moved J1 4.97 mm to (1.90, 22.2), turned to 90 degrees
- moved J3 2.15 mm to (19.2, 25.5)
Routing:
- net GND: track 199.5 -> 168.0 mm, vias 5 -> 23
- net Q1_GATE: track 58.0 -> 37.7 mm, vias 2 -> 0
- net BUS_CLAMP: track 41.4 -> 28.9 mm
- net NRST: track 90.2 -> 84.1 mm, vias 5 -> 3
- net SWCLK: track 51.3 -> 56.0 mm, vias 3 -> 6
- net VBAT_RAW: track 55.2 -> 58.8 mm
- net VBAT: track 79.3 -> 82.3 mm, vias 2 -> 3
- net BUS_DATA: track 49.1 -> 49.3 mm, vias 5 -> 6

Commit message: sync: 2026-10-15 日常更新
Parts:
- added R17: 0R, R_0603_1608Metric, F.Cu at (18.8, 6.35)
- moved C1 10.6 mm to (23.5, 29.0)
Routing:
- net VBAT: track 82.3 -> 100.7 mm, vias 3 -> 5
- net SWCLK: track 56.0 -> 54.0 mm
- net GND: vias 23 -> 27

Commit message: sync: 2026-10-15 日常更新
Routing:
- net VBAT: track 100.7 -> 106.3 mm
- net GND: vias 27 -> 37
Changed lines of the file:
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@@
 	)
 	(segment
+		(start 36.96 19.78)
+		(end 36.2 20.5)
+		(width 0.25)
+		(layer "B.Cu")
+		(net "VBAT")
+	)
+	(segment
+		(start 38.2 21)
+		(end 36.2 20.5)
+		(width 0.25)
+		(layer "B.Cu")
+		(net "VBAT")
+	)
+	(segment
 		(start 35.7 13.04)
 		(end 36.9561 14.2961)
@@
 	)
 	(segment
+		(start 36.2 20.5)
+		(end 35.7 21.04)
+		(width 0.25)
+		(layer "B.Cu")
+		(net "VBAT")
+	)
+	(segment
 		(start 38.2 21)
 		(end 38.3 22.4)
@@
 	)
 	(segment
+		(start 36 13.2)
+		(end 35.7 13.04)
+		(width 0.25)
+		(layer "B.Cu")
+		(net "VBAT")
+	)
+	(segment
 		(start 14.6 11)
 		(end 15.8277 12.2277)
@@
 	)
 	(segment
+		(start 36.96 14.3)
+		(end 36 13.2)
+		(width 0.25)
+		(layer "B.Cu")
+		(net "VBAT")
+	)
+	(segment
 		(start 18.08 12.2277)
 		(end 18.5541 11.7536)
@@
 	)
 	(via
+		(at 3 15)
+		(size 0.7)
+		(drill 0.35)
+		(layers "F.Cu" "B.Cu")
+		(net "GND")
+	)
+	(via
 		(at 29.08 7.46)
 		(size 0.7)
@@
 	)
 	(via
+		(at 29 8.5)
+		(size 0.7)
+		(drill 0.35)
+		(layers "F.Cu" "B.Cu")
+		(net "GND")
+	)
+	(via
+		(at 3 9.5)
+		(size 0.7)
+		(drill 0.35)
+		(layers "F.Cu" "B.Cu")
+		(net "GND")
+	)
+	(via
 		(at 12.35 25.34)
 		(size 0.7)
@@
 	)
 	(via
+		(at 27 20)
+		(size 0.7)
+		(drill 0.35)
+		(layers "F.Cu" "B.Cu")
+		(net "GND")
+	)
+	(via
 		(at 16.3771 20.2729)
 		(size 0.7)
@@
 	)
 	(via
+		(at 17.5 22.5)
+		(size 0.7)
+		(drill 0.35)
+		(layers "F.Cu" "B.Cu")
+		(net "GND")
+	)
+	(via
 		(at 22.02 23.45)
 		(size 0.7)
@@
 	)
 	(via
+		(at 13 10)
+		(size 0.7)
+		(drill 0.35)
+		(layers "F.Cu" "B.Cu")
+		(net "GND")
+	)
+	(via
 		(at 27.53 17.73)
 		(size 0.7)
@@
 	)
 	(via
+		(at 21 8.5)
+		(size 0.7)
+		(drill 0.35)
+		(layers "F.Cu" "B.Cu")
+		(net "GND")
+	)
+	(via
+		(at 3 9)
+		(size 0.7)
+		(drill 0.35)
+		(layers "F.Cu" "B.Cu")
+		(net "GND")
+	)
+	(via
 		(at 11.73 1.5)
 		(size 0.7)
@@
 	)
 	(via
+		(at 4 8.5)
+		(size 0.7)
+		(drill 0.35)
+		(layers "F.Cu" "B.Cu")
+		(net "GND")
+	)
+	(via
 		(at 23.6 24.34)
 		(size 0.7)
@@
 	)
 	(via
+		(at 3 8.5)
+		(size 0.7)
+		(drill 0.35)
+		(layers "F.Cu" "B.Cu")
+		(net "GND")
+	)
+	(via
 		(at 4 7.5)
 		(size 0.7)
@@
 			(thermal_gap 0.5)
 			(thermal_bridge_width 0.5)
-			(island_removal_mode 2)
-			(island_area_min 2)
+			(island_removal_mode 0)
 		)
 		(polygon
@@
 			(thermal_gap 0.5)
 			(thermal_bridge_width 0.5)
-			(island_removal_mode 2)
-			(island_area_min 2)
+			(island_removal_mode 0)
 		)
 		(polygon

Commit message: sync: 2026-10-15 日常更新
Parts:
- C14: moved to B.Cu
- J1: value BattPad_1x02_P3.6 -> BATT IN 2.54 2P
- R17: value 0R -> 0R (jumper)
- moved R16 28.3 mm to (15.3, 7.03)
- moved C13 16.5 mm to (22.0, 20.8)
- moved R7 15.3 mm to (35.8, 27.5)
- moved C14 12.0 mm to (8.50, 21.0), turned to 0 degrees
- moved C11 11.1 mm to (13.5, 20.3)
- moved C1 9.64 mm to (17.8, 21.2)
- moved R9 6.14 mm to (10.0, 20.8)
- moved J2 5.18 mm to (4.60, 19.9)
- moved R17 4.73 mm to (23.0, 4.28), turned to 0 degrees
- moved R5 4.42 mm to (11.3, 16.3)
- moved R6 3.78 mm to (14.8, 11.0)
- moved C7 3.75 mm to (15.3, 9.03)
- moved J1 3.10 mm to (1.90, 25.3)
- moved C12 2.00 mm to (38.3, 7.53)
- moved R8 2.00 mm to (38.3, 5.53)
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Connections:
- C2 pad 1: VBAT -> VBAT_C2
- R17 pad 2: VBAT -> VBAT_C2
Routing:
- net RX_EN: track 26.8 -> 95.4 mm, vias 2 -> 5
- net GND: track 168.0 -> 218.7 mm, vias 37 -> 4
- net SWDIO: track 23.0 -> 60.1 mm, vias 1 -> 2
- net OCS_AUX: track 14.3 -> 47.1 mm, vias 2 -> 8
- net VBAT: track 106.3 -> 74.1 mm, vias 5 -> 2
- net SWCLK: track 54.0 -> 80.3 mm, vias 6 -> 9
- net UART1_TX: track 57.2 -> 80.3 mm, vias 3 -> 4
- net UART1_RX: track 44.7 -> 63.0 mm, vias 4 -> 5
- net BUS_TX: track 22.2 -> 37.5 mm, vias 1 -> 2
- net BUS_CLAMP: track 28.9 -> 42.5 mm, vias 1 -> 3
- net SCx: track 16.9 -> 29.9 mm
- net VBAT_RAW: track 58.8 -> 46.5 mm
- net +3V3: track 129.6 -> 118.5 mm, vias 3 -> 4
- net BUS_LOGIC: track 52.5 -> 41.9 mm, vias 1 -> 5
- net BUS_DATA: track 49.3 -> 57.8 mm, vias 6 -> 1
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- added copper zone on B.Cu, net VBAT

Commit message: sync: 2026-10-15 日常更新
Parts:
- U3: footprint TSSOP-8_3x3mm_P0.65mm -> VSSOP-8_2.3x2mm_P0.5mm
- moved R16 29.0 mm to (35.8, 27.5)
- moved R7 13.4 mm to (23.3, 22.8)
- moved C13 3.75 mm to (25.8, 20.8)
- moved R14 3.64 mm to (26.5, 24.8)
- moved R15 1.50 mm to (26.5, 26.8)
- moved R3 1.35 mm to (26.8, 22.8)
- moved C1 1.25 mm to (19.1, 21.2)
- moved C11 1.25 mm to (14.8, 20.3)
- moved R9 1.25 mm to (11.3, 20.8)
- moved U3 0.65 mm to (31.1, 21.6), turned to 180 degrees
Routing:
- net RX_EN: track 95.4 -> 30.5 mm, vias 5 -> 0
- net NRST: track 89.6 -> 35.0 mm, vias 9 -> 3
- net GND: track 218.7 -> 175.5 mm
- net OCS_AUX: track 47.1 -> 12.7 mm, vias 8 -> 2
- net UART1_TX: track 80.3 -> 47.4 mm, vias 4 -> 0
- net SWCLK: track 80.3 -> 57.6 mm, vias 9 -> 0
- net VBAT: track 74.1 -> 95.7 mm, vias 2 -> 3
- net VBAT_LOGIC: track 74.1 -> 52.8 mm, vias 6 -> 4
- net SCx: track 29.9 -> 9.81 mm, vias 2 -> 0
- net BUS_CLAMP: track 42.5 -> 27.0 mm, vias 3 -> 1
- net BUS_DATA: track 57.8 -> 47.8 mm, vias 1 -> 0
- net IMU_INT2: track 20.2 -> 10.9 mm
- net V3V3_IMU: track 61.7 -> 52.9 mm, vias 10 -> 3
- net SPI_MISO: track 23.3 -> 14.6 mm, vias 4 -> 2
- net UART1_RX: track 63.0 -> 54.4 mm, vias 5 -> 0
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